Commit message: best i was able to do

File: arm.urdf (robot description, URDF)
Before this commit: robot robot, 4 links, 3 joints
Joints:
- joint 2: limit lower=-3.14159 upper=0 effort=0.0 velocity=0.0 -> lower=-3.14159 upper=3.14 effort=0.0 velocity=0.0

Commit message: i tried :(

File: arm.urdf (robot description, URDF)
Before this commit: robot robot, 4 links, 3 joints
Joints:
- joint 1: limit lower=-3.14159 upper=0 effort=0.0 velocity=0.0 -> lower=-6.28318 upper=6.28318 effort=0.0 velocity=0.0
- joint 2: limit lower=-3.14159 upper=3.14 effort=0.0 velocity=0.0 -> lower=-6.28318 upper=6.28318 effort=0.0 velocity=0.0
- joint 3: limit lower=-3.14159 upper=3.14159 effort=0.0 velocity=0.0 -> lower=-6.28318 upper=6.28318 effort=0.0 velocity=0.0

Commit message: new ver

File: arm.urdf (robot description, URDF)
Before this commit: robot robot, 4 links, 3 joints
Joints:
- joint 1: limit lower=-6.28318 upper=6.28318 effort=0.0 velocity=0.0 -> lower=-2.3561924999999997 upper=2.3561924999999997 effort=0.0 velocity=0.0
- joint 2: limit lower=-6.28318 upper=6.28318 effort=0.0 velocity=0.0 -> lower=-2.3561924999999997 upper=2.3561924999999997 effort=0.0 velocity=0.0
- joint 3: limit lower=-6.28318 upper=6.28318 effort=0.0 velocity=0.0 -> lower=-2.3561924999999997 upper=2.3561924999999997 effort=0.0 velocity=0.0
